File: colorimeter-2.kicad_sch (KiCad schematic)
At the start: 47 parts, among them IC1 MAX1561ETA+T, IC2 MAX1561ETA+T, IC3 MAX1561ETA+T, J1 Full15_Female, J2 Full15_Male, J3 D_Photo_Filled, J4 D_Photo_Filled, J5 LED_RGB, J6 LED_RGB

Commit message: MAX4583 switch between LED groups + amp decoupling caps
Parts:
- removed C10, C11, C7, C8, C9: C, Capacitor_SMD:C_0805_2012Metric_Pad1.18x1.45mm_HandSolder, symbol Device:C
- removed D1, D2, D3: D_Schottky, Diode_SMD:D_0805_2012Metric_Pad1.15x1.40mm_HandSolder, symbol Device:D_Schottky
- removed IC1, IC2, IC3: MAX1561ETA+T, SamacSys_Parts:SON65P300X300X80-9N, symbol SamacSys_Parts:MAX1561ETA+T
- removed L1, L2, L3: L, mylib:L_Bourns_CC322522A, symbol Device:L
- removed R7, R8, R9: R, Resistor_SMD:R_0805_2012Metric_Pad1.20x1.40mm_HandSolder, symbol Device:R
- added IC1: MAX4583, SamacSys_Parts:SOIC127P600X175-16N, symbol mylib:MAX4583
- C3, C5: value C -> 10uF
- C4, C6: value C -> 0.1uF
Connections:
- net 0: now also IC1.11 (A)
- net 1: now also IC1.10 (B)
- net 2: now also IC1.9 (C)
- net GND: now also C3.2, C4.2, C5.1, IC1.8 (GND); no longer C3.1, C4.1, C5.2
- net V+: now also C3.1, C4.1, IC1.16 (V_{CC}), IC1.6 (ENABLE); no longer C4.2, C6.2
- net V-: now also C5.2, C6.2, IC1.7 (V_{EE})
- net at J5.1 (RK): now also IC1.3 (Z1); no longer J6.6 (RA)
- net at J5.2 (GK): now also IC1.1 (Y1); no longer J6.5 (GA)
- net at J5.3 (BK): now also IC1.13 (X1); no longer J6.4 (BA)
- net CurrentSense_B: no longer names the net of J6.3 (BK)
- net CurrentSense_B: now also IC1.12 (X0)
- net CurrentSense_G: no longer names the net of J6.2 (GK)
- net CurrentSense_G: now also IC1.2 (Y0)
- net CurrentSense_R: no longer names the net of J6.1 (RK)
- net CurrentSense_R: now also IC1.5 (Z0)
- net LEDPower_B: no longer names the net of J5.4 (BA)
- net LEDPower_G: no longer names the net of J5.5 (GA)
- net LEDPower_R: no longer names the net of J5.6 (RA)
- net LEDPower_R: no longer C5.1
Other:
- note added: "WIP under-constant-change LED driver circuit:"
- note removed: "LED Drivers"
- moved on the sheet: C1, J3, J5, J6, JP3, JP4, NT1, R1, R2, R3, U1A, U1C
